File: workspace/switch_and_amplifiers/rx_lna_preamp/preamp.kicad_pcb (KiCad board)
At the start: 2 copper layers, 40 x 24 mm, 25 parts, among them J1 RF_IN, J2 RF_OUT, J3 Power, U1 PHA-13LN, U2 7805

Commit message: Order at JLCPCB with modified rf clearances
Parts:
- C7: value 100n,16V,20% -> 100n,50V,10%
Routing:
- net GND: track 94.4 -> 89.6 mm
Other:
- board text added: "@20MHz"
- board text added: "G=24dB"
- board text added: "JLCJLCJLCJLC"
- board text added: "N=1.2dB"
