File: workspace/rx_lna_preamp/preamp.kicad_pcb (KiCad board)
At the start: 2 copper layers, 40 x 24 mm, 25 parts, among them J1 RF_IN, J2 RF_OUT, J3 Power, U1 PHA-13LN, U2 7805

Commit message: Update file permissions, rf_switch and poweramp
Parts:
- removed the G*** at (161.6, 83.7)
Other:
- board text added: "IN"
- board text added: "OUT"
- board text added: "P1dB=23dBm"
- board text added: "Pin=6dBm max"
