File: workspace/tr_switch/tr_switch.kicad_sch (KiCad schematic)
At the start: 18 parts, among them J1 RF1, J2 RF2, J2 RFC, J3 Control, J3 Power, U2 7805, U2 QPC6324

Commit message: Get TR-Switch Rev 1 ready for ordering
Parts:
- C5: MPN (none) -> CL21B105KBFNNNG; Mouser 80-C0805C104J5R -> 187-CL21B105KBFNNNG
- C5: MPN (none) -> C0805C201K5HACTU; Mouser (none) -> 80-C0805C201K5HACTU
- C8, C9: value 1u,50V,10% -> 1u/50V
- J3: MPN 68491-102HLF -> 69190-104HLF; Mouser 649-68491-102HLF -> 649-69190-104HLF
- U2: footprint tr_switch:QFN-20-1EP_4x4mm_P0.5mm_EP2x2mm_HandSolder -> Package_DFN_QFN:QFN-20-1EP_4x4mm_P0.5mm_EP2.5x2.5mm_ThermalVias; Mouser (none) -> 772-QPC6324TR13
Changed lines of the file:
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@@
       (effects (font (size 1.27 1.27)) (justify left))
     )
-    (property "Value" "1u,50V,10%" (at 91.2368 43.053 0)
+    (property "Value" "1u/50V" (at 91.2368 43.053 0)
       (effects (font (size 1.27 1.27)) (justify left))
     )
@@
       (effects (font (size 1.27 1.27)))
     )
-    (property "Footprint" "tr_switch:QFN-20-1EP_4x4mm_P0.5mm_EP2x2mm_HandSolder" (at 138.43 92.71 0)
+    (property "Footprint" "Package_DFN_QFN:QFN-20-1EP_4x4mm_P0.5mm_EP2.5x2.5mm_ThermalVias" (at 138.43 92.71 0)
       (effects (font (size 1.27 1.27)) hide)
     )
@@
       (effects (font (size 1.27 1.27)) hide)
     )
-    (property "Mouser" "" (at 138.684 113.03 0)
-      (effects (font (size 1.27 1.27)))
+    (property "Mouser" "772-QPC6324TR13" (at 139.7 127 0) (do_not_autoplace)
+      (effects (font (size 1.27 1.27)) hide)
     )
     (pin "1")
@@
     (pin "19")
     (pin "2")
-    (pin "2")
     (pin "20")
     (pin "21")
@@
       (effects (font (size 1.27 1.27)) (justify left))
     )
-    (property "Value" "1u,50V,10%" (at 54.4068 43.053 0)
+    (property "Value" "1u/50V" (at 54.4068 43.053 0)
       (effects (font (size 1.27 1.27)) (justify left))
     )
@@
       (effects (font (size 1.27 1.27)) hide)
     )
-    (property "Datasheet" " ~" (at 163.83 113.03 0)
+    (property "Datasheet" "https://www.farnell.com/datasheets/2048997.pdf" (at 163.83 113.03 0)
       (effects (font (size 1.27 1.27)) hide)
     )
@@
       (effects (font (size 1.27 1.27)) hide)
     )
-    (property "Datasheet" "~" (at 133.35 67.31 0)
-      (effects (font (size 1.27 1.27)) hide)
-    )
-    (property "MPN" "68491-102HLF " (at 133.35 67.31 0)
-      (effects (font (size 1.27 1.27)) hide)
-    )
-    (property "Mouser" "649-68491-102HLF" (at 133.35 67.31 0)
+    (property "Datasheet" "https://cdn.amphenol-cs.com/media/wysiwyg/files/documentation/datasheet/boardwiretoboard/bwb_bergstik.pdf" (at 133.35 67.31 0)
+      (effects (font (size 1.27 1.27)) hide)
+    )
+    (property "MPN" "69190-104HLF" (at 133.35 67.31 0)
+      (effects (font (size 1.27 1.27)) hide)
+    )
+    (property "Mouser" "649-69190-104HLF" (at 133.35 67.31 0)
       (effects (font (size 1.27 1.27)) hide)
     )
@@
       (effects (font (size 1.27 1.27)) hide)
     )
-    (property "Datasheet" "~" (at 147.32 97.79 0)
-      (effects (font (size 1.27 1.27)) hide)
-    )
-    (property "MPN" "" (at 147.32 97.79 90)
-      (effects (font (size 1.27 1.27)) hide)
-    )
-    (property "Mouser" "80-C0805C104J5R" (at 147.32 97.79 90)
+    (property "Datasheet" "https://www.mouser.ch/datasheet/2/585/MLCC-1837944.pdf" (at 147.32 97.79 0)
+      (effects (font (size 1.27 1.27)) hide)
+    )
+    (property "MPN" "CL21B105KBFNNNG" (at 147.32 97.79 90)
+      (effects (font (size 1.27 1.27)) hide)
+    )
+    (property "Mouser" "187-CL21B105KBFNNNG" (at 147.32 97.79 90)
       (effects (font (size 1.27 1.27)) hide)
     )
@@
       (effects (font (size 1.27 1.27)) hide)
     )
-    (property "Datasheet" "~" (at 127 97.79 0)
-      (effects (font (size 1.27 1.27)) hide)
-    )
-    (property "MPN" "" (at 127 97.79 90)
-      (effects (font (size 1.27 1.27)) hide)
-    )
-    (property "Mouser" "" (at 127 97.79 90)
+    (property "Datasheet" "https://www.mouser.ch/datasheet/2/212/KEM_C1007_X8R_ULTRA_150C_SMD-1102703.pdf" (at 127 97.79 0)
+      (effects (font (size 1.27 1.27)) hide)
+    )
+    (property "MPN" "C0805C201K5HACTU" (at 127 97.79 90)
+      (effects (font (size 1.27 1.27)) hide)
+    )
+    (property "Mouser" "80-C0805C201K5HACTU" (at 127 97.79 90)
       (effects (font (size 1.27 1.27)) hide)
     )
@@
       (effects (font (size 1.27 1.27)) hide)
     )
-    (property "Datasheet" "~" (at 147.32 86.36 0)
+    (property "Datasheet" "https://www.mouser.ch/datasheet/2/212/KEM_C1002_X7R_SMD-1102033.pdf" (at 147.32 86.36 0)
       (effects (font (size 1.27 1.27)) hide)
     )
@@
       (effects (font (size 1.27 1.27)) hide)
     )
-    (property "Datasheet" " ~" (at 138.43 138.43 0)
+    (property "Datasheet" "https://www.farnell.com/datasheets/2048997.pdf" (at 138.43 138.43 0)
       (effects (font (size 1.27 1.27)) hide)
     )
@@
       (effects (font (size 1.27 1.27)) hide)
     )
-    (property "Datasheet" "~" (at 127 86.36 0)
-      (effects (font (size 1.27 1.27)) hide)
-    )
-    (property "MPN" "" (at 127 86.36 90)
-      (effects (font (size 1.27 1.27)) hide)
-    )
-    (property "Mouser" "" (at 127 86.36 90)
+    (property "Datasheet" "https://www.mouser.ch/datasheet/2/212/KEM_C1007_X8R_ULTRA_150C_SMD-1102703.pdf" (at 127 86.36 0)
+      (effects (font (size 1.27 1.27)) hide)
+    )
+    (property "MPN" "C0805C201K5HACTU" (at 127 86.36 90)
+      (effects (font (size 1.27 1.27)) hide)
+    )
+    (property "Mouser" "80-C0805C201K5HACTU" (at 127 86.36 90)
       (effects (font (size 1.27 1.27)) hide)
     )
@@
       (effects (font (size 1.27 1.27)) hide)
     )
-    (property "Datasheet" "~" (at 24.13 38.1 0)
-      (effects (font (size 1.27 1.27)) hide)
-    )
+    (property "Datasheet" "https://cdn.amphenol-cs.com/media/wysiwyg/files/documentation/datasheet/boardwiretoboard/bwb_bergstik.pdf" (at 24.13 38.1 0)
+      (effects (font (size 1.27 1.27)) hide)
+    )
