File: workspace/tx_power_amp/poweramp.kicad_pcb (KiCad board)
At the start: 2 copper layers, 76 x 37 mm, 54 parts, among them J1 Power, J2 RF_IN, J3 RF_OUT, J4 Power_Enable, Q1 MMBT3904, Q2 BCP51, U1 ADL5536, U2 PHA-202+, U3 LM317_SOT-223, U4 LM317_SOT-223

Commit message: Get poweramp Rev 1 ready for ordering
Other:
- board text added: "JLCJLCJLCJLC"
