File: workspace/tx_power_amp/poweramp.kicad_sch (KiCad schematic)
At the start: 53 parts, among them J1 RF_IN, J2 RF_OUT, J3 Power, J3 Power_Enable, Q1 2N3904, Q2 BCP51, U1 ADL5536, U2 PHA-202+, U3 LM317_SOT-223, U4 LM317_SOT-223

Commit message: Update file permissions, rf_switch and poweramp
Parts:
- Q1: value 2N3904 -> MMBT3904; footprint Package_TO_SOT_THT:TO-92_Inline -> Package_TO_SOT_SMD:SOT-23; MPN (none) -> MMBT3904-7-F; Mouser (none) -> 621-MMBT3904-F
- R11: value 1k -> 4k7
- R9: value 1k -> 10k
- U2: footprint poweramp:DL1636 -> poweramp:DL1636_HandSolder
Connections:
- net GND: now also U2.1 (EP), U2.3 (EP), U2.4 (EP), U2.5 (EP), U2.6 (EP), U2.8 (EP)
- net att_in: now reaches C2.2, R1.1, R3.1
- net amp_in: now reaches C3.2, U2.2
- net amp_out: now reaches C4.1, L1.2, U2.7
- net preamp_out: now reaches C2.1, L2.2, U1.3
- net filter_out: now reaches C1.1, C19.2, L3.2
- net preamp_in: now reaches C1.2, U1.1
- net att_out: now reaches C3.1, R2.1, R3.2
Other:
- company: (none) -> ETH Zürich
- title: (none) -> RF Power Amplifier
Changed lines of the file:
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@@
 (kicad_sch (version 20230121) (generator eeschema)
   (paper "A4")
+  (title_block
+    (title "RF Power Amplifier")
+    (date "2023-06-23")
+    (rev "1")
+    (company "ETH Zürich")
+    (comment 1 "Maximilian Stabel")
+  )
   (junction (at 102.87 172.72) (diameter 0) (color 0 0 0 0)
   )
@@
     (effects (font (size 1.27 1.27)) (justify left bottom))
   )
+  (label "preamp_out" (at 132.08 76.2 0) (fields_autoplaced)
+    (effects (font (size 1.27 1.27)) (justify left bottom))
+  )
+  (label "amp_in" (at 193.04 76.2 0) (fields_autoplaced)
+    (effects (font (size 1.27 1.27)) (justify left bottom))
+  )
+  (label "att_out" (at 172.72 76.2 0) (fields_autoplaced)
+    (effects (font (size 1.27 1.27)) (justify left bottom))
+  )
+  (label "amp_out" (at 234.95 76.2 0) (fields_autoplaced)
+    (effects (font (size 1.27 1.27)) (justify left bottom))
+  )
+  (label "att_in" (at 156.21 76.2 0) (fields_autoplaced)
+    (effects (font (size 1.27 1.27)) (justify left bottom))
+  )
   (label "rf_out" (at 255.27 76.2 0) (fields_autoplaced)
     (effects (font (size 1.27 1.27)) (justify left bottom))
   )
+  (label "preamp_in" (at 93.98 76.2 0) (fields_autoplaced)
+    (effects (font (size 1.27 1.27)) (justify left bottom))
+  )
+  (label "filter_out" (at 73.66 76.2 0) (fields_autoplaced)
+    (effects (font (size 1.27 1.27)) (justify left bottom))
+  )
   (label "rf_in" (at 27.94 76.2 0) (fields_autoplaced)
     (effects (font (size 1.27 1.27)) (justify left bottom))
@@
   (symbol (lib_id "Device:R") (at 227.33 132.08 180) (unit 1)
     (in_bom yes) (on_board yes) (dnp no) (fields_autoplaced)
-    (property "Reference" "R10" (at 229.8262 130.81 0)
+    (property "Reference" "R10" (at 229.87 130.81 0)
       (effects (font (size 1.27 1.27)) (justify right))
     )
-    (property "Value" "1k" (at 229.8262 133.35 0)
+    (property "Value" "1k" (at 229.87 133.35 0)
       (effects (font (size 1.27 1.27)) (justify right))
     )
@@
   (symbol (lib_id "Device:R") (at 227.33 121.92 180) (unit 1)
     (in_bom yes) (on_board yes) (dnp no) (fields_autoplaced)
-    (property "Reference" "R11" (at 229.8262 120.65 0)
+    (property "Reference" "R11" (at 229.87 120.65 0)
       (effects (font (size 1.27 1.27)) (justify right))
     )
-    (property "Value" "1k" (at 229.8262 123.19 0)
+    (property "Value" "4k7" (at 229.87 123.19 0)
       (effects (font (size 1.27 1.27)) (justify right))
     )
@@
       (effects (font (size 1.27 1.27)) (justify left))
     )
-    (property "Value" "2N3904" (at 229.87 143.51 0)
-      (effects (font (size 1.27 1.27)) (justify left))
-    )
-    (property "Footprint" "Package_TO_SOT_THT:TO-92_Inline" (at 229.87 144.145 0)
+    (property "Value" "MMBT3904" (at 229.87 143.51 0)
+      (effects (font (size 1.27 1.27)) (justify left))
+    )
+    (property "Footprint" "Package_TO_SOT_SMD:SOT-23" (at 229.87 144.145 0)
       (effects (font (size 1.27 1.27) italic) (justify left) hide)
     )
-    (property "Datasheet" "https://www.onsemi.com/pub/Collateral/2N3903-D.PDF" (at 224.79 142.24 0)
+    (property "Datasheet" "https://www.mouser.ch/datasheet/2/115/DIOD_S_A0003133141_1-2542424.pdf" (at 224.79 142.24 0)
       (effects (font (size 1.27 1.27)) (justify left) hide)
     )
+    (property "MPN" "MMBT3904-7-F" (at 224.79 142.24 0)
+      (effects (font (size 1.27 1.27)) hide)
+    )
+    (property "Mouser" "621-MMBT3904-F" (at 224.79 142.24 0)
+      (effects (font (size 1.27 1.27)) hide)
+    )
     (pin "1")
     (pin "2")
@@
       (effects (font (size 1.27 1.27)))
     )
-    (property "Footprint" "poweramp:DL1636" (at 215.9 66.04 0)
+    (property "Footprint" "poweramp:DL1636_HandSolder" (at 215.9 66.04 0)
       (effects (font (size 1.27 1.27)) hide)
     )
@@
       (effects (font (size 1.27 1.27)) hide)
     )
-    (pin "2")
+    (pin "1")
+    (pin "2")
+    (pin "3")
+    (pin "4")
+    (pin "5")
+    (pin "6")
     (pin "7")
+    (pin "8")
     (pin "EP")
     (instances
@@
       (effects (font (size 1.27 1.27)) (justify right))
     )
-    (property "Value" "1k" (at 220.9362 148.59 0)
+    (property "Value" "10k" (at 220.9362 148.59 0)
       (effects (font (size 1.27 1.27)) (justify right))
     )

Commit message: Get poweramp Rev 1 ready for ordering
Parts:
- C1, C10, C15, C2, C3, C4: Notes (none) -> 10%
- C11, C5: MPN (none) -> CL21B105KBFNNNG; Mouser 80-C0805C104J5R -> 187-CL21B105KBFNNNG; Notes (none) -> 10%
- C12, C6: MPN (none) -> 08055C102KAT2A; Mouser 80-C0805C104J5R -> 581-08055C102K; Notes (none) -> 10%
- C18, C19: MPN (none) -> GRM2165C1H131JA01D; Mouser (none) -> 81-GRM215C1H131JA01D
- C7: MPN (none) -> 08055A680JAT2A; Mouser 80-C0805C104J5R -> 581-08055A680J
- C8, C9: value 1u,50V,10% -> 1u/50V; Notes (none) -> 10%
- L3: MPN (none) -> 36502AR36JTDG; Mouser (none) -> 279-36502AR36JTDG; Notes (none) -> 5%,RF
- Q2: MPN (none) -> BCP51,115; Mouser (none) -> 771-BCP51115
- R1, R2: MPN (none) -> AC0805FR-07150RL; Mouser (none) -> 603-AC0805FR-07150RL
- R10, R8: MPN (none) -> 1623131-1; Mouser (none) -> 279-1623131-1
- R11: MPN (none) -> AC0805FR-074K7L; Mouser (none) -> 603-AC0805FR-074K7L
- R3: MPN (none) -> CR0805-FX-37R4ELF; Mouser (none) -> 652-CR0805FX-37R4ELF
- R9: MPN (none) -> CRCW080510K0FKEAC; Mouser (none) -> 71-CRCW080510K0FKEAC
- U1: MPN (none) -> ADL5536ARKZ-R7; Mouser (none) -> 584-ADL5536ARKZ-R7
- U2: MPN (none) -> PHA-202+; Mouser (none) -> 139-PHA-202
