File: workspace/32-channel_current_source/32-channel_current_source/32-channel_current_source.kicad_sch (KiCad schematic)
At the start: 16 parts, among them U1 LM4040DBZ-2.5, U3 LM317_SOT-223, U4 LM337_SOT223

Commit message: Update 32-Channel Current Source Rev 1
Parts:
- removed C1, C2: 1000u/25V, symbol Device:C_Polarized_Small
- removed C3, C4: 22u/50V, symbol Device:C_Polarized_Small
- removed C5: 470u/50V, symbol Device:C_Polarized_Small
- removed D1, D2, D3, D4: MRA4003T3G, Diode_SMD:D_SMA, symbol Diode:MRA4003T3G
- removed R1, R2: 1k8, symbol Device:R_Small
- removed R3, R4: 1, symbol Device:R_Small
- removed U1: LM4040DBZ-2.5, Package_TO_SOT_SMD:SOT-23, symbol Reference_Voltage:LM4040DBZ-2.5
- removed U3: LM317_SOT-223, Package_TO_SOT_SMD:SOT-223-3_TabPin2, symbol Regulator_Linear:LM317_SOT-223
- removed U4: LM337_SOT223, Package_TO_SOT_SMD:SOT-223-3_TabPin2, symbol Regulator_Linear:LM337_SOT223
- added H1, H2, H3, H4: MountingHole_Pad, MountingHole:MountingHole_3.2mm_M3_Pad_Via, symbol Mechanical:MountingHole_Pad
- added J1, J2, J3: Conn_01x01, Connector:CalTest_CT3151, symbol Connector_Generic:Conn_01x01
- added J4: Conn_02x05_Odd_Even, Connector_IDC:IDC-Header_2x05_P2.54mm_Vertical_SMD, symbol Connector_Generic:Conn_02x05_Odd_Even
Connections:
- net GND: now also H1.1, H2.1, H3.1, H4.1, J2.1 (Pin_1), J4.10 (Pin_10), J4.2 (Pin_2), J4.4 (Pin_4), J4.6 (Pin_6), J4.8 (Pin_8)
- net VCC: now also J4.1 (Pin_1)
- net VEE: now also J3.1 (Pin_1)
- new net CS: J4.9 (Pin_9)
- new net MISO: J4.5 (Pin_5)
- new net MOSI: J4.3 (Pin_3)
- new net SCLK: J4.7 (Pin_7)
- new net VDD: J1.1 (Pin_1)
Other:
- added sheet 8-channel_current_source (8-channel_current_source.kicad_sch)
- added sheet 8-channel_current_source1 (8-channel_current_source.kicad_sch)
- added sheet 8-channel_current_source2 (8-channel_current_source.kicad_sch)
- added sheet 8-channel_current_source3 (8-channel_current_source.kicad_sch)
- note added: "Alternating GND/Signal on IDC Cable => Simple Shield"
- note added: "Daisy-Chain Operation"
- note added: "Main Power 2.7V..3.3V 16A"
- note added: "SPI Power 1.62V..5.5V"
- note added: "TODO: Galvanic Isolation?"
- note removed: "10V"
- note removed: "From https://www.diyaudio.com/community/threads/virtual-ground-a-regulated-rail-splitter.234665/"
- note removed: "Set R_{1}/R_{2} for current of 2mA"
- company: (none) -> ETH Zürich
- title: (none) -> 32-Channel Programmable Current Source

Commit message: Finish Rev 1 of the 32-channel current supply
Parts:
- added H5, H6: MountingHole_Pad, MountingHole:MountingHole_6.4mm_M6_ISO14580_Pad, symbol Mechanical:MountingHole_Pad
- added N1: Hammond 1590, symbol Mechanical:Housing_Pad
- H1, H2, H3, H4: footprint MountingHole:MountingHole_3.2mm_M3_Pad_Via -> MountingHole:MountingHole_6.4mm_M6_ISO14580_Pad; now left out of the parts list
- J1: footprint Connector:CalTest_CT3151 -> Connector_Wire:SolderWirePad_1x01_SMD_5x10mm; Enclosure-Datasheet (none) -> https://www.mouser.ch/datasheet/2/215/091-744596.pdf; Enclosure-MPN (none) -> 6091; Enclosure-Mouser (none) -> 534-6091; MPN CT3151-2 -> (none); Mouser 510-CT3151-2 -> (none)
- J2: footprint Connector:CalTest_CT3151 -> Connector_Wire:SolderWirePad_1x01_SMD_5x10mm; Enclosure-Datasheet (none) -> https://www.mouser.ch/datasheet/2/215/092-743448.pdf; Enclosure-MPN (none) -> 6092; Enclosure-Mouser (none) -> 534-6092; MPN CT3151-0 -> (none); Mouser 510-CT3151-0 -> (none)
- J3: footprint Connector:CalTest_CT3151 -> Connector_Wire:SolderWirePad_1x01_SMD_5x10mm; Enclosure-Datasheet (none) -> https://www.mouser.ch/datasheet/2/215/091-744596.pdf; Enclosure-MPN (none) -> 6091; Enclosure-Mouser (none) -> 534-6091; MPN CT3151-0 -> (none); Mouser 510-CT3151-0 -> (none); now left out of the parts list
- J4: Enclosure-Datasheet (none) -> https://www.mouser.ch/datasheet/2/1/7f640c6e18f1d8480b1473b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; Enclosure-MPN (none) -> 4610-6000; Enclosure-Mouser (none) -> 517-4610-6000; MPN (none) -> 72454-010LF; Mouser (none) -> 649-72454-010LF; Notes (none) -> 10 pos, 2 row, DIN41651, 2.54mm PCB pitch, 1.27mm cable pit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; Receptacle-Datasheet (none) -> https://cdn.amphenol-cs.com/media/wysiwyg/files/documentati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; Receptacle-MPN (none) -> 71600-310LF; Receptacle-Mouser (none) -> 649-71600-310LF
Connections:
- net GND: now also H5.1, H6.1, N1.1 (PAD)
Other:
- note added: "+2.7V..+3.3V GND -2.7V..-3.3V 16A"
- note added: "Current Sources"
- note added: "Daisy-Chained SPI Operation"
- note added: "Don't forget the cables inside the enclosure"
- note added: "Enclosure"
- note added: "For connectors see "Enclosure-*" entries"
- note added: "Mounting Holes"
- note added: "Power Connector"
- note added: "SPI"
- note added: "Used for cooling as well"
- note removed: "Daisy-Chain Operation"
- note removed: "Main Power 2.7V..3.3V 16A"
- moved on the sheet: H1, H2, H3, H4, J4
