File: workspace/32-channel_current_source/32-channel_current_source/8-channel_current_source.kicad_sch (KiCad schematic)
At the start: 6 parts, among them J1 Conn_02x08_Odd_Even, U4 AD5676R

Commit message: Finish Rev 1 of the 32-channel current supply
Parts:
- J1: DigiKey S9187-ND -> (none); Enclosure-Datasheet (none) -> https://www.mouser.ch/datasheet/2/1/7cf9f07a304787bc0d985f8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; Enclosure-MPN (none) -> 4616-6000; Enclosure-Mouser (none) -> 517-4616-6000; MPN SBH11-NBPC-D08-SM-BK -> 72454-016LF; Mouser (none) -> 649-72454-016LF; Notes (none) -> 16 pos, 2 row, DIN41651, 2.54mm PCB pitch, 1.27mm cable pit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; Receptacle-Datasheet (none) -> https://cdn.amphenol-cs.com/media/wysiwyg/files/documentati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; Receptacle-MPN (none) -> 71600-316LF; Receptacle-Mouser (none) -> 649-71600-316LF
- U4: MPN (none) -> AD5676RBRUZ; Mouser (none) -> 584-AD5676RBRUZ
Other:
- note added: "Coil Connector (8x)"
- note added: "DAC"
- note added: "U-I-Converters"
- moved on the sheet: J1
