File: hardware/transmit_power_amplifier/poweramp.kicad_sch (KiCad schematic)
At the start: 53 parts, among them J1 RF_IN, J2 RF_OUT, J3 Power, J3 Power_Enable, Q1 MMBT3904, Q2 BCP51, U1 ADL5536, U2 PHA-202+, U3 LM317_SOT-223, U4 LM317_SOT-223

Commit message: Add 3D models for 3D render
Parts:
- F2: Manufacturer Littelfuse -> (none); Mouser (none) -> 576-0805L075SLYR
Changed lines of the file:
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@@
-      (effects (font (size 1.27 1.27)) hide)
-    )
-    (property "Manufacturer" "Littelfuse" (at 29.21 123.19 0)
       (effects (font (size 1.27 1.27)) hide)
     )
@@
       (effects (font (size 1.27 1.27)) hide)
     )
+    (property "Mouser" "576-0805L075SLYR" (at 29.21 123.19 90)
+      (effects (font (size 1.27 1.27)) hide)
+    )
