File: hardware/receive_preamplifier/preamp.kicad_sch (KiCad schematic)
At the start: 23 parts, among them J1 RF_IN, J2 RF_OUT, J3 Power, U1 PHA-13LN, U2 7805

Commit message: Fix lna feedback loop
Parts:
- C3: footprint Capacitor_SMD:C_0805_2012Metric -> Capacitor_SMD:C_0402_1005Metric_Pad0.74x0.62mm_HandSolder; MPN CL21B104KBCNNNC -> GRM155R71H104KE14D; Mouser 187-CL21B104KBCNNNC -> 81-GRM155R71H104KE4D
- R1: footprint Resistor_SMD:R_0805_2012Metric -> Resistor_SMD:R_0402_1005Metric_Pad0.72x0.64mm_HandSolder; MPN RT0805FRE101K5L -> RC0402FR-071K5L; Mouser 603-RT0805FRE101K5L -> 603-RC0402FR-071K5L
Changed lines of the file:
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@@
       (effects (font (size 1.27 1.27)))
     )
-    (property "Footprint" "Capacitor_SMD:C_0805_2012Metric" (at 140.97 125.73 0)
+    (property "Footprint" "Capacitor_SMD:C_0402_1005Metric_Pad0.74x0.62mm_HandSolder" (at 140.97 125.73 0)
       (effects (font (size 1.27 1.27)) hide)
     )
-    (property "Datasheet" "https://www.mouser.ch/datasheet/2/585/MLCC-1837944.pdf" (at 140.97 125.73 0)
+    (property "Datasheet" "https://www.mouser.ch/datasheet/2/281/1/GRM155R71H104KE14_01A-1984472.pdf" (at 140.97 125.73 0)
       (effects (font (size 1.27 1.27)) hide)
     )
-    (property "MPN" "CL21B104KBCNNNC" (at 140.97 125.73 90)
+    (property "MPN" "GRM155R71H104KE14D" (at 140.97 125.73 90)
       (effects (font (size 1.27 1.27)) hide)
     )
-    (property "Mouser" "187-CL21B104KBCNNNC" (at 140.97 125.73 90)
+    (property "Mouser" "81-GRM155R71H104KE4D" (at 140.97 125.73 90)
       (effects (font (size 1.27 1.27)) hide)
     )
@@
       (effects (font (size 1.27 1.27)))
     )
-    (property "Footprint" "Resistor_SMD:R_0805_2012Metric" (at 152.4 125.73 0)
+    (property "Footprint" "Resistor_SMD:R_0402_1005Metric_Pad0.72x0.64mm_HandSolder" (at 152.4 125.73 0)
       (effects (font (size 1.27 1.27)) hide)
     )
-    (property "Datasheet" "https://www.mouser.ch/datasheet/2/447/PYu_RT_1_to_0_01_RoHS_L_12-3003070.pdf" (at 152.4 125.73 0)
+    (property "Datasheet" "https://www.mouser.ch/datasheet/2/447/YAGEO_PYu_RC_Group_51_RoHS_L_12-3313492.pdf" (at 152.4 125.73 0)
       (effects (font (size 1.27 1.27)) hide)
     )
-    (property "MPN" "RT0805FRE101K5L" (at 152.4 125.73 90)
+    (property "MPN" "RC0402FR-071K5L" (at 152.4 125.73 90)
       (effects (font (size 1.27 1.27)) hide)
     )
-    (property "Mouser" "603-RT0805FRE101K5L" (at 152.4 125.73 90)
+    (property "Mouser" "603-RC0402FR-071K5L" (at 152.4 125.73 90)
       (effects (font (size 1.27 1.27)) hide)
     )
